File: schematics/1500WRMS-VCGA-CLASS-H-AUDIO-POWER-AMPLIFIER-NS-LAB-VERSION/1500WRMS-VCGA-CLASS-H-AUDIO-POWER-AMPLIFIER-NS-LAB-VERSION.sch (KiCad schematic (older format))
At the start: 208 parts, among them Q401 2N5551, Q402 2N5551, Q403 2N5551, Q404 MJE340, Q405 MJE350, Q406 MJE350, Q407 MJE350, Q408 2N5551, Q409 MJE340, Q501 2N5401, Q502 MJE350, Q503 2N5551, Q504 MJE340, Q505 MJE340, Q506 MJE15032, Q507 2SC5200, Q5081 2SC5200, Q50810 2SC5200, Q50811 2SC5200, Q5082 2SC5200, Q5083 2SC5200, Q5084 2SC5200, Q5085 2SC5200, Q5086 2SC5200, Q5087 2SC5200, Q5088 2SC5200, Q5089 2SC5200, Q509 MJE15033, Q510 2SA1943, Q511 2SA1943, Q5111 2SA1943, Q51110 2SA1943, Q51111 2SA1943, Q5113 2SA1943, Q5114 2SA1943, Q5115 2SA1943, Q5116 2SA1943, Q5117 2SA1943, Q5118 2SA1943, Q5119 2SA1943, Q512 2N5551, Q513 2N5401, Q601 2N5551, Q602 2N5401, Q603 2N5401, Q604 2N5401, Q605 2N5551, Q606 2N5551, X6011 IRF9540, X6012 IRF9540, X6021 IRF540, X6022 IRF540

Commit message: Commit Wed May  8 11:35:14 UTC 2019
Parts:
- added C301, C702: 10uF, VCGA:CAPACITOR_AE_D10mm, symbol VCGA:CAPACITOR_ELECTROLYTE
- added C302: 220uF, VCGA:CAPACITOR_AE_D10mm, symbol VCGA:CAPACITOR_ELECTROLYTE
- added C701: 1uF, VCGA:CAPACITOR_AE_D10mm, symbol VCGA:CAPACITOR_ELECTROLYTE
- added D301, D302: 1N4738, VCGA:DIODE_AXIAL_SMALL_SI, symbol VCGA:ZENER
- added D303, D304, D701, D702, D703, D704, D705, D706: 1N4148, VCGA:DIODE_AXIAL_SMALL_GE, symbol VCGA:DIODE
- added D707: 1N4732, VCGA:DIODE_AXIAL_SMALL_SI, symbol VCGA:ZENER
- added D708: 1N4002, VCGA:DIODE_AXIAL_SMALL_SI, symbol VCGA:DIODE
- added Q301, Q701, Q703, Q704: 2N5551, VCGA:TO-92-EBC, symbol VCGA:Q_NPN
- added Q702: 2N5401, VCGA:TO-92-EBC, symbol VCGA:Q_PNP
- added Q705: TIP42C, VCGA:DIODE_POWER_TO-220, symbol VCGA:Q_PNP
- added R301, R701, R702: 100k, VCGA:RESISTOR_AXIAL_0.25W, symbol VCGA:RESISTOR
- added R302: 3.3k, VCGA:RESISTOR_AXIAL_0.25W, symbol VCGA:RESISTOR
- added R303, R703, R711: 1k, VCGA:RESISTOR_AXIAL_0.25W, symbol VCGA:RESISTOR
- added R304: 180k, VCGA:RESISTOR_AXIAL_0.25W, symbol VCGA:RESISTOR
- added R305, R307, R309: 100k, VCGA:RESISTOR_AXIAL_0.5W, symbol VCGA:RESISTOR
- added R306, R308, R310, R312, R708, R709, R710, R712: 2.7k, VCGA:RESISTOR_AXIAL_0.25W, symbol VCGA:RESISTOR
- added R311, R714: 15k, VCGA:RESISTOR_AXIAL_0.25W, symbol VCGA:RESISTOR
- added R704: 4.7k, VCGA:RESISTOR_AXIAL_0.25W, symbol VCGA:RESISTOR
- added R705: 120k, VCGA:RESISTOR_AXIAL_0.25W, symbol VCGA:RESISTOR
- added R706, R707: 10k, VCGA:RESISTOR_AXIAL_0.25W, symbol VCGA:RESISTOR
- added R713: 2.2k, VCGA:RESISTOR_AXIAL_0.25W, symbol VCGA:RESISTOR
- added R715: 12k, VCGA:RESISTOR_AXIAL_0.25W, symbol VCGA:RESISTOR
- added R716: 82k, VCGA:RESISTOR_AXIAL_0.25W, symbol VCGA:RESISTOR
- added R717: 5.6k, VCGA:RESISTOR_AXIAL_0.25W, symbol VCGA:RESISTOR
- added R718: 3.9k, VCGA:RESISTOR_AXIAL_0.25W, symbol VCGA:RESISTOR
- added R719: 150, VCGA:RESISTOR_AXIAL_1W, symbol VCGA:RESISTOR
- added XLOC301: NSL32, VCGA:NSL32, symbol VCGA:LDR_OPTO_COUPLER
- added XOC701: PC817, VCGA:DIP4, symbol VCGA:OPTO_COUPLER
- added XU301, XU302, XU701: JRC4558, VCGA:DIP8, symbol VCGA:JRC4558
- R603, R604, R612, R613: value 12k -> 15k
Connections:
- net 0: now also C302.2, C701.2, C702.2, D304.1 (A), D701.1 (A), D702.2 (K), D703.2 (K), D704.1 (A), Q301.3 (E), Q703.3 (E), R301.2, R304.2, R306.2, R308.2, R310.2, R703.2, R707.2, R708.1, R709.2, R715.2, R717.2, XLOC301.4, XOC701.3
- net M_INPUT: now also C301.1; no longer C401.1
- net M_VSWON: now also R619.1; no longer R619.2
- net M_VSWOP: now also R619.2; no longer R619.1
- net M_OUT_RAW: now reaches D601.1 (A), D608.2 (K), L501.1, Q512.3 (E), Q513.3 (E), R403.1, R510.2, R511.1, R5121.2, R51210.2, R51211.2, R5122.2, R5123.2, R5124.2, R5125.2, R5126.2, R5127.2, R5128.2, R5129.2, R5131.1, R51310.1, R51311.1, R5132.1, R5133.1, R5134.1, R5135.1, R5136.1, R5137.1, R5138.1, R5139.1, R517.1, R519.1, R520.1
- net M_OUT_RAW: now also R305.1, R701.1
- net M_FPSSP: now reaches R5141.2, R51410.2, R51411.2, R5142.2, R5143.2, R5144.2, R5145.2, R5146.2, R5147.2, R5148.2, R5149.2, R516.2
- net M_FPSSP: now also D707.2 (K)
- net M_FPSSN: now reaches R5151.1, R51510.1, R51511.1, R5152.1, R5153.1, R5154.1, R5155.1, R5156.1, R5157.1, R5158.1, R5159.1, R518.2
- net M_FPSSN: now also XOC701.2
- net M_VCCHN renamed -120V
- net -120V: now also D302.1 (A)
- net M_VCCHP renamed +120V
- net +120V: now also D301.2 (K)
- net M_VCCLN renamed -42V
- net M_VCCLP renamed +42V
- new net: C401.1, R303.1, XU301.7 (OUT)
- new net: R302.1, XU301.1 (OUT), XU301.2 (-)
- new net: C301.2, R301.1, XU301.3 (+)
- new net: R302.2, XLOC301.3, XU301.5 (+)
- new net: R303.2, R304.1, XU301.6 (-)
- new net: D701.2 (K), D702.1 (A), R701.2, XU701.3 (+)
- new net: D304.2 (K), Q301.2 (B), R311.2
- new net: D301.1 (A), R307.1
- new net: D303.1 (A), R307.2, R308.1, XU302.6 (-)
- new net: C701.1, R705.2, XU701.5 (+)
- new net: R706.2, R707.1, XU701.6 (-)
- new net: R702.1, R704.1, XU701.1 (OUT)
- new net: R305.2, R306.1, XU302.3 (+), XU302.5 (+)
- new net: D302.2 (K), R309.1
- new net: R309.2, R310.1, XU302.2 (-)
- new net: R312.2, XLOC301.1
- new net: D707.1 (A), R711.1
- new net: R711.2, XOC701.1
- new net: R712.2, XOC701.4
- new net: Q702.2 (B), R710.2, R712.1, R713.2
- new net: Q704.3 (E), R717.1
- new net: Q704.1 (C), Q705.2 (B), R718.2
- new net: Q702.1 (C), R714.1
- new net: R702.2, R703.1, XU701.2 (-)
- new net: D706.1 (A), Q701.3 (E), R709.1
- new net: D705.2 (K), Q701.2 (B), R708.2
- new net: Q701.1 (C), R710.1
- new net +15V: Q702.3 (E), Q705.3 (E), R312.1, R713.1, R716.1, R718.1, XU301.8 (VCC), XU301.8 (VCC), XU302.8 (VCC), XU302.8 (VCC), XU701.8 (VCC), XU701.8 (VCC)
- new net +RLC: D708.2 (K), Q705.1 (C)
- new net -15V: R719.2, XU301.4 (VEE), XU301.4 (VEE), XU302.4 (VEE), XU302.4 (VEE), XU701.4 (VEE), XU701.4 (VEE)
- new net -RLC: D708.1 (A), R719.1
- new net LIMIT_IND_SRC: C302.1, Q301.1 (C), XLOC301.2
- new net M_FPODLO: D703.1 (A), D704.2 (K), R704.2, R705.1
- new net M_FPODO: D705.1 (A), D706.2 (K), R706.1, XU701.7 (OUT)
- new net M_FPSO: Q703.2 (B), R714.2, R715.1
- new net M_FPTH: C702.1, Q703.1 (C), Q704.2 (B), R716.2
- new net M_LMSON: D303.2 (K), XU302.1 (OUT)
- new net M_LMSOP: R311.1, XU302.7 (OUT)
Other:
- note added: "DC V. supply in\n+120V"
- note added: "DC V. supply in\n+15V"
- note added: "DC V. supply in\n+42V"
- note added: "DC V. supply in\n-120V"
- note added: "DC V. supply in\n-15V"
- note added: "DC V. supply in\n-42V"
- note added: "FAULT / SHORT & OPEN CIRCUIT PROTECTION"
- note added: "INPUT:\n1V RMS NOM.\n10V RMS MAX.\n"
- note added: "LIMITER"
- note added: "SINK-SIDE STEPPER"
- note added: "TECHNICAL NOTICE:\nThe resistors without wattage specification are 0.25W.\nApply only capacitor with working voltage specification\nat 250V or above for C404 and C405 to prevent\nunexpected output DC slewing in stationer state."
- note added: "To limit indicator\namplifier input"
- note added: "To protector\nrelay +NC"
- note added: "To protector\nrelay coil"
- note added: "UNITY CURRENT\nGAIN & POWER\nAMPLIFICATION\nSTAGE"
- note added: "UP-SIDE STEPPER"
- note added: "VOLTAGE GAIN\nAMPLIFICATION\nSTAGE"
- note removed: "DC V. SUPPLY IN\n+120V"
- note removed: "DC V. SUPPLY IN\n+42V"
- note removed: "DC V. SUPPLY IN\n-120V"
- note removed: "DC V. SUPPLY IN\n-42V"
- note removed: "INPUT FROM\nLOW IMPEDANCE\nSOURCE AT\n1V RMS MAX."
- note removed: "TECHNICAL NOTICE:\nThe resistors without wattage specification are 0.25W. Apply only\ncapacitor with working voltage specification at 250V or above for\nC404 and C405 to prevent unexpected output DC slewing in sta-\ntioner state."
- moved on the sheet: C401, C402, C403, C404, C405, C501, C502, C601, C602, C603, C604, D401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

Commit message: Commit Wed May  8 12:11:19 UTC 2019
Parts:
- C301, C701, C702: footprint VCGA:CAPACITOR_AE_D10mm -> VCGA:CAPACITOR_AE_D7.62mm
- C401, C403: Voltage 100V -> 50V
- Q705: footprint VCGA:DIODE_POWER_TO-220 -> VCGA:TO-220
Changed lines of the file:
@@
 F 0 "C301" V 1200 8950 50  0000 C CNN
 F 1 "10uF" V 1100 9100 50  0000 C CNN
-F 2 "VCGA:CAPACITOR_AE_D10mm" H 1350 8950 50  0001 C CNN
+F 2 "VCGA:CAPACITOR_AE_D7.62mm" H 1350 8950 50  0001 C CNN
 F 3 "" H 1350 8950 50  0001 C CNN
 F 4 "16V" V 1100 8900 50  0000 C CNN "Voltage"
@@
 F 0 "C702" H 13950 8950 50  0000 C CNN
 F 1 "10uF" H 13950 8850 50  0000 C CNN
-F 2 "VCGA:CAPACITOR_AE_D10mm" H 14150 8850 50  0001 C CNN
+F 2 "VCGA:CAPACITOR_AE_D7.62mm" H 14150 8850 50  0001 C CNN
 F 3 "" H 14150 8850 50  0001 C CNN
 F 4 "16V" H 13950 8750 50  0000 C CNN "Voltage"
@@
 F 0 "Q705" H 15000 8400 50  0000 C CNN
 F 1 "TIP42C" H 15000 8500 50  0000 C CNN
-F 2 "VCGA:DIODE_POWER_TO-220" H 14800 8450 50  0001 C CNN
+F 2 "VCGA:TO-220" H 14800 8450 50  0001 C CNN
 F 3 "" H 14800 8450 50  0001 C CNN
 F 4 "Q" H 15750 8400 50  0001 C CNN "Spice_Primitive"
@@
 F 0 "C701" H 10050 8850 50  0000 C CNN
 F 1 "1uF" H 10050 8750 50  0000 C CNN
-F 2 "VCGA:CAPACITOR_AE_D10mm" H 10250 8750 50  0001 C CNN
+F 2 "VCGA:CAPACITOR_AE_D7.62mm" H 10250 8750 50  0001 C CNN
 F 3 "" H 10250 8750 50  0001 C CNN
 F 4 "16V" H 10050 8650 50  0000 C CNN "Voltage"
@@
 F 2 "VCGA:CAPACITOR_AE_D10mm" H 3050 4550 50  0001 C CNN
 F 3 "" H 3050 4550 50  0001 C CNN
-F 4 "100V" H 3250 4450 50  0000 C CNN "Voltage"
+F 4 "50V" H 3250 4450 50  0000 C CNN "Voltage"
 	1    3050 4550
 	1    0    0    -1
@@
 F 2 "VCGA:CAPACITOR_AE_D10mm" H 1850 6400 50  0001 C CNN
 F 3 "" H 1850 6400 50  0001 C CNN
-F 4 "100V" H 1650 6500 50  0000 C CNN "Voltage"
+F 4 "50V" H 1650 6500 50  0000 C CNN "Voltage"
 	1    1850 6400
 	-1   0    0    1
@@
 	9850 9050 9850 9150
 $Comp
-L pspice:0 #GND?
+L pspice:0 #GND0105
 U 1 1 6081DBF4
 P 9850 9450
-F 0 "#GND?" H 9850 9350 50  0001 C CNN
+F 0 "#GND0105" H 9850 9350 50  0001 C CNN
 F 1 "0" H 9850 9537 50  0001 C CNN
 F 2 "" H 9850 9450 50  0001 C CNN

Commit message: Commit Thu May  9 11:52:12 UTC 2019
Parts:
- added R305: 100k, VCGA:RESISTOR_AXIAL_0.5W, symbol VCGA:RESISTOR
- added R310: 2.7k, VCGA:RESISTOR_AXIAL_0.25W, symbol VCGA:RESISTOR
- renumbered R305 to R309, R309 to R311, R310 to R312, R311 to R313, R312 to R314
Connections:
- net 0: now also R310.2
- net M_OUT_RAW: now also R305.1
- net at R306.1, XU302.5 (+): now also R305.2; no longer R309.2, XU302.3 (+)
- new net: R309.2, R310.1, XU302.3 (+)
Other:
- moved on the sheet: D301, R307, R311, XU302A
Changed lines of the file:
@@
 EESchema Schematic File Version 4
-LIBS:1500WRMS-VCGA-CLASS-H-AUDIO-POWER-AMPLIFIER-NS-LAB-VERSION-cache
+LIBS:ANALYSIS-1500WRMS-VCGA-CLASS-H-AUDIO-POWER-AMPLIFIER-NS-LAB-VERSION-cache
 EELAYER 29 0
 EELAYER END
 $Descr A3 16535 11693
 encoding utf-8
-Sheet 1 1
+Sheet 2 2
 Title "1500W RMS Class-H Audio Power Amplifier Core Circuit"
 Date "2019-05-08"
@@
 	1    0    0    -1
 $EndComp
-Text Label 5300 9050 3    40   ~ 0
+Text Label 5300 9000 3    40   ~ 0
 M_LMSON
 Connection ~ 4950 9650
 Wire Wire Line
-	4950 9150 4950 9650
+	4950 9100 4950 9650
 Wire Wire Line
-	5250 8950 5300 8950
+	5250 8900 5300 8900
 Wire Wire Line
 	4450 8250 4450 8400
@@
 	4450 9400 4450 9450
 Wire Wire Line
-	4450 8700 4450 8600
+	4450 8650 4450 8600
 $Comp
 L pspice:0 #GND0116
@@
 L VCGA:ZENER D301
 U 1 1 646B338B
-P 5700 8250
-F 0 "D301" V 5550 8250 50  0000 C CNN
-F 1 "1N4738" V 5450 8250 50  0000 C CNN
-F 2 "VCGA:DIODE_AXIAL_SMALL_SI" H 5700 8250 50  0001 C CNN
-F 3 "" H 5700 8250 50  0001 C CNN
-F 4 "D" H 6650 8200 50  0001 C CNN "Spice_Primitive"
-F 5 "Y" H 6650 8100 50  0001 C CNN "Spice_Netlist_Enabled"
-F 6 "spice_models/model.lib" H 6650 8400 50  0001 C CNN "Spice_Lib_File"
-F 7 "1N4738" H 5700 8250 50  0001 C CNN "Spice_Model"
-	1    5700 8250
+P 5850 8250
+F 0 "D301" V 5700 8250 50  0000 C CNN
+F 1 "1N4738" V 5600 8250 50  0000 C CNN
+F 2 "VCGA:DIODE_AXIAL_SMALL_SI" H 5850 8250 50  0001 C CNN
+F 3 "" H 5850 8250 50  0001 C CNN
+F 4 "D" H 6800 8200 50  0001 C CNN "Spice_Primitive"
+F 5 "Y" H 6800 8100 50  0001 C CNN "Spice_Netlist_Enabled"
+F 6 "spice_models/model.lib" H 6800 8400 50  0001 C CNN "Spice_Lib_File"
+F 7 "1N4738" H 5850 8250 50  0001 C CNN "Spice_Model"
+	1    5850 8250
 	0    -1   -1   0
 $EndComp
@@
 L VCGA:JRC4558 XU302
 U 1 1 60E6D2CA
-P 4950 8950
-F 0 "XU302" H 4700 8650 50  0000 C CNN
-F 1 "JRC4558" H 4700 8550 50  0000 C CNN
-F 2 "VCGA:DIP8" H 4950 8950 50  0001 C CNN
-F 3 "" H 4950 8950 50  0001 C CNN
-F 4 "X" H 4950 8950 50  0001 C CNN "Spice_Primitive"
-F 5 "RC4558_IMPL" H 4950 8950 50  0001 C CNN "Spice_Model"
-F 6 "Y" H 4950 8950 50  0001 C CNN "Spice_Netlist_Enabled"
-F 7 "spice_models/model.lib" H 4950 8950 50  0001 C CNN "Spice_Lib_File"
-	1    4950 8950
+P 4950 8900
+F 0 "XU302" H 5200 9250 50  0000 C CNN
+F 1 "JRC4558" H 5200 9150 50  0000 C CNN
+F 2 "VCGA:DIP8" H 4950 8900 50  0001 C CNN
+F 3 "" H 4950 8900 50  0001 C CNN
+F 4 "X" H 4950 8900 50  0001 C CNN "Spice_Primitive"
+F 5 "RC4558_IMPL" H 4950 8900 50  0001 C CNN "Spice_Model"
+F 6 "Y" H 4950 8900 50  0001 C CNN "Spice_Netlist_Enabled"
+F 7 "spice_models/model.lib" H 4950 8900 50  0001 C CNN "Spice_Lib_File"
+	1    4950 8900
 	1    0    0    -1
 $EndComp
@@
 $EndComp
 $Comp
-L VCGA:RESISTOR R312
+L VCGA:RESISTOR R314
 U 1 1 6A08C3EB
 P 2550 8650
-F 0 "R312" H 2600 8700 50  0000 L CNN
+F 0 "R314" H 2600 8700 50  0000 L CNN
 F 1 "2.7k" H 2600 8600 50  0000 L CNN
 F 2 "VCGA:RESISTOR_AXIAL_0.25W" H 2550 8650 50  0001 C CNN
@@
 Connection ~ 6050 8900
 Wire Wire Line
-	6050 8900 5900 8900
-Wire Wire Line
 	2900 8400 2950 8400
 Wire Wire Line
@@
 	2950 8400 3250 8400
 Wire Wire Line
-	4650 8850 4600 8850
+	4650 8800 4600 8800
 Wire Wire Line
-	4450 9000 4450 9050
+	4450 8950 4450 9000
 Wire Wire Line
-	4450 9050 4650 9050
-Connection ~ 4450 9050
+	4450 9000 4650 9000
+Connection ~ 4450 9000
 Wire Wire Line
-	4450 9050 4450 9100
+	4450 9000 4450 9100
 Connection ~ 5450 8700
 Wire Wire Line
-	5300 8950 5300 9500
+	5300 8900 5300 9500
 Wire Wire Line
-	5800 8250 5900 8250
+	5950 8250 6050 8250
 Wire Wire Line
-	5900 8250 5900 8350
+	6050 8250 6050 8300
 Wire Wire Line
 	2550 9400 2550 9800
@@
 Connection ~ 3550 8050
 Wire Wire Line
-	4950 8750 4950 8050
+	4950 8700 4950 8050
 Connection ~ 4950 8050
 Wire Wire Line
@@
 Text Notes 3800 9550 0    75   ~ 0
 LIMITER
-Text GLabel 5500 8250 0    50   Input ~ 0
+Text GLabel 5650 8250 0    50   Input ~ 0
 +120V
 Wire Wire Line
-	5600 8250 5500 8250
-Wire Wire Line
-	5900 8650 5900 8900
-Connection ~ 5900 8900
-Wire Wire Line
-	5900 8900 5750 8900
+	5750 8250 5650 8250
 Text GLabel 7250 8500 2    50   Output ~ 0
 LIMIT_IND_SRC
@@
 Text Label 6850 9100 1    40   ~ 0
 M_LMSOP
-Wire Wire Line
-	4600 8400 4600 8500
-Wire Wire Line
-	4600 8500 5450 8500
-Connection ~ 4600 8500
-Wire Wire Line
-	4600 8500 4600 8850
-Wire Wire Line
-	5450 8500 5450 8700
 $Comp
-L VCGA:RESISTOR R311
+L VCGA:RESISTOR R313
 U 1 1 5DD4F556
 P 7050 9150
-F 0 "R311" V 7250 9150 50  0000 C CNN
+F 0 "R313" V 7250 9150 50  0000 C CNN
 F 1 "15k" V 7150 9150 50  0000 C CNN
 F 2 "VCGA:RESISTOR_AXIAL_0.25W" H 7050 9150 50  0001 C CNN
@@
 $EndComp
 $Comp
-L VCGA:RESISTOR R310
+L VCGA:RESISTOR R312
 U 1 1 60E6D2D4
 P 4450 9250
-F 0 "R310" H 4250 9300 50  0000 C CNN
+F 0 "R312" H 4250 9300 50  0000 C CNN
 F 1 "2.7k" H 4250 9200 50  0000 C CNN
 F 2 "VCGA:RESISTOR_AXIAL_0.25W" H 4450 9250 50  0001 C CNN
@@
 $EndComp
 $Comp
-L VCGA:RESISTOR R309
+L VCGA:RESISTOR R311
 U 1 1 60E6D2E4
-P 4450 8850
-F 0 "R309" H 4250 8950 50  0000 C CNN
-F 1 "100k" H 4250 8850 50  0000 C CNN
-F 2 "VCGA:RESISTOR_AXIAL_0.5W" H 4450 8850 50  0001 C CNN
-F 3 "" H 4450 8850 50  0001 C CNN
-F 4 "0.5W" H 4250 8750 50  0000 C CNN "Wattage"
-	1    4450 8850
+P 4450 8800
+F 0 "R311" H 4250 8900 50  0000 C CNN
+F 1 "100k" H 4250 8800 50  0000 C CNN
+F 2 "VCGA:RESISTOR_AXIAL_0.5W" H 4450 8800 50  0001 C CNN
+F 3 "" H 4450 8800 50  0001 C CNN
+F 4 "0.5W" H 4250 8700 50  0000 C CNN "Wattage"
+	1    4450 8800
 	1    0    0    -1
 $EndComp
 $Comp
-L VCGA:RESISTOR R305
+L VCGA:RESISTOR R309
 U 1 1 6079E951
 P 4600 8250
-F 0 "R305" H 4750 8350 50  0000 C CNN
+F 0 "R309" H 4750 8350 50  0000 C CNN
 F 1 "100k" H 4750 8250 50  0000 C CNN
 F 2 "VCGA:RESISTOR_AXIAL_0.5W" H 4600 8250 50  0001 C CNN
@@
 L VCGA:RESISTOR R307
 U 1 1 5EEE4D35
-P 5900 8500
-F 0 "R307" H 6050 8600 50  0000 C CNN
-F 1 "100k" H 6050 8500 50  0000 C CNN
-F 2 "VCGA:RESISTOR_AXIAL_0.5W" H 5900 8500 50  0001 C CNN
-F 3 "" H 5900 8500 50  0001 C CNN
-F 4 "0.5W" H 6050 8400 50  0000 C CNN "Wattage"
-	1    5900 8500
+P 6050 8450
+F 0 "R307" H 6200 8550 50  0000 C CNN
+F 1 "100k" H 6200 8450 50  0000 C CNN
+F 2 "VCGA:RESISTOR_AXIAL_0.5W" H 6050 8450 50  0001 C CNN
+F 3 "" H 6050 8450 50  0001 C CNN
+F 4 "0.5W" H 6200 8350 50  0000 C CNN "Wattage"
+	1    6050 8450
 	1    0    0    -1
 $EndComp
@@
 	11100 8650 11050 8650
 Wire Wire Line
-	4600 7900 8600 7900
+	4600 7900 5050 7900
 Wire Wire Line
 	8600 8100 8600 7900
@@
 	9850 9050 9850 9150
 $Comp
-L pspice:0 #GND0105
+L pspice:0 #GND0135
 U 1 1 6081DBF4
 P 9850 9450
-F 0 "#GND0105" H 9850 9350 50  0001 C CNN
+F 0 "#GND0135" H 9850 9350 50  0001 C CNN
 F 1 "0" H 9850 9537 50  0001 C CNN
 F 2 "" H 9850 9450 50  0001 C CNN
@@
 Wire Wire Line
 	9850 9350 9850 9450
+Wire Wire Line
+	5750 8900 6050 8900
+Wire Wire Line
+	6050 8600 6050 8900
+$Comp
+L VCGA:RESISTOR R305
+U 1 1 5D2086DA
+P 5050 8250
+F 0 "R305" H 5200 8350 50  0000 C CNN
+F 1 "100k" H 5200 8250 50  0000 C CNN
+F 2 "VCGA:RESISTOR_AXIAL_0.5W" H 5050 8250 50  0001 C CNN
+F 3 "" H 5050 8250 50  0001 C CNN
+F 4 "0.5W" H 5200 8150 50  0000 C CNN "Wattage"
+	1    5050 8250
+	1    0    0    -1
+$EndComp
+Wire Wire Line
+	5050 8100 5050 7900
+Connection ~ 5050 7900
+Wire Wire Line
+	5050 7900 8600 7900
+$Comp
+L VCGA:RESISTOR R310
+U 1 1 5D46E172
+P 4600 9250
+F 0 "R310" H 4650 9300 50  0000 L CNN
+F 1 "2.7k" H 4650 9200 50  0000 L CNN
+F 2 "VCGA:RESISTOR_AXIAL_0.25W" H 4600 9250 50  0001 C CNN
+F 3 "" H 4600 9250 50  0001 C CNN
+	1    4600 9250
+	1    0    0    -1
+$EndComp
+Wire Wire Line
+	5050 8400 5050 8450
+Wire Wire Line
+	5050 8450 5450 8450
+Wire Wire Line
+	5450 8450 5450 8700
+$Comp
+L pspice:0 #GND0136
+U 1 1 5D6DAD1D
+P 4600 9450
+F 0 "#GND0136" H 4600 9350 50  0001 C CNN
+F 1 "0" H 4600 9537 50  0001 C CNN
+F 2 "" H 4600 9450 50  0001 C CNN
+F 3 "~" H 4600 9450 50  0001 C CNN
+	1    4600 9450
+	1    0    0    -1
+$EndComp
+Wire Wire Line
+	4600 9450 4600 9400
+Wire Wire Line
+	4600 8400 4600 8800
+Connection ~ 4600 8800
+Wire Wire Line
+	4600 8800 4600 9100
 $EndSCHEMATC

Commit message: Commit Mon May 13 03:19:53 UTC 2019
Parts:
- R4011: value 300 -> 330
- R605, R614, R701: footprint VCGA:RESISTOR_AXIAL_0.25W -> VCGA:RESISTOR_AXIAL_0.5W; Wattage (none) -> 0.5W
- X6011, X6012, X6021, X6022: footprint VCGA:TO-220 -> VCGA:TO-220-MIRRORED
- renumbered Q511 to Q5112
Connections:
- net 0: now also D701.2 (K), D702.1 (A); no longer D701.1 (A), D702.2 (K)
- net M_REF: now also R4011.1, R4012.1; no longer R4011.2, R4012.2
- net at R701.2, XU701.3 (+): now also D701.1 (A), D702.2 (K); no longer D701.2 (K), D702.1 (A)
- new net: C401.2, R4011.2, R4012.2
Other:
- moved on the sheet: C401, C402, C403, D401, D701, Q401, Q402, Q403, Q404, Q407, Q408, R402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
