File: schematics/1500WRMS-VCGA-CLASS-H-AUDIO-POWER-AMPLIFIER-NS-LAB-VERSION/1500WRMS-VCGA-CLASS-H-AUDIO-POWER-AMPLIFIER-NS-LAB-VERSION.sch (KiCad schematic (older format))
At the start: 268 parts, among them Q301 2N5551, Q401 2N5551, Q402 2N5551, Q403 2N5551, Q404 MJE340, Q405 MJE350, Q406 MJE350, Q407 MJE350, Q408 2N5551, Q409 MJE340, Q501 2N5401, Q502 MJE350, Q503 2N5551, Q504 MJE340, Q505 MJE340, Q506 MJE15032, Q507 2SC5200, Q5081 2SC5200, Q50810 2SC5200, Q50811 2SC5200, Q5082 2SC5200, Q5083 2SC5200, Q5084 2SC5200, Q5085 2SC5200, Q5086 2SC5200, Q5087 2SC5200, Q5088 2SC5200, Q5089 2SC5200, Q509 MJE15033, Q510 2SA1943, Q5111 2SA1943, Q51110 2SA1943, Q51111 2SA1943, Q5112 2SA1943, Q5113 2SA1943, Q5114 2SA1943, Q5115 2SA1943, Q5116 2SA1943, Q5117 2SA1943, Q5118 2SA1943, Q5119 2SA1943, Q512 2N5551, Q513 2N5401, Q601 2N5551, Q602 2N5401, Q603 2N5401, Q604 2N5401, Q605 2N5551, Q606 2N5551, Q701 2N5551, Q702 2N5401, Q703 2N5551, Q704 2N5551, Q705 TIP42C, X6011 IRF9540, X6012 IRF9540, X6021 IRF540, X6022 IRF540

Commit message: Commit Wed May 15 20:03:55 UTC 2019
Parts:
- added R720: 100k, VCGA:RESISTOR_AXIAL_0.5W, symbol VCGA:RESISTOR
- added SR701: sw1 ON, VCGA:RL-SLA24, symbol VCGA:RELAY_STD
Connections:
- net +RLC: now also SR701.3
- net -RLC: now also SR701.4
- net 0: now also R720.2
- net M_OUT: now also SR701.2; no longer L501.2
- new net: L501.2, R720.1, SR701.1
Other:
- note added: "To SPEAKER\nTERMINAL (+)"
- note removed: "To protector\nrelay +NC"
- note removed: "To protector\nrelay coil"
Changed lines of the file:
@@
 EESchema Schematic File Version 4
-LIBS:1500WRMS-VCGA-CLASS-H-AUDIO-POWER-AMPLIFIER-NS-LAB-VERSION-cache
+LIBS:ANALYSIS-1500WRMS-VCGA-CLASS-H-AUDIO-POWER-AMPLIFIER-NS-LAB-VERSION-cache
 EELAYER 29 0
 EELAYER END
 $Descr A3 16535 11693
 encoding utf-8
-Sheet 1 1
+Sheet 2 2
 Title "1500W RMS Class-H Audio Power Amplifier Core Circuit"
 Date "2019-05-13"
@@
 Text GLabel 7050 6400 0    50   Input ~ 0
 -42V
-Text GLabel 15550 7900 2    50   Output ~ 0
+Text GLabel 15550 9300 2    50   Output ~ 0
 M_OUT
-Text HLabel 15700 4900 0    50   BiDi ~ 0
+Text HLabel 15450 9150 2    50   BiDi ~ 0
 M_OUT
 Text HLabel 7800 800  0    50   BiDi ~ 0
@@
 $EndComp
 Wire Wire Line
-	14800 8850 14800 8800
-Wire Wire Line
 	14800 9600 14800 9650
-Wire Wire Line
-	14800 8800 14950 8800
-Connection ~ 14800 8800
-Wire Wire Line
-	14800 8800 14800 8650
-Text GLabel 14950 8800 2    50   Output ~ 0
-+RLC
-Text GLabel 14950 9100 2    50   Output ~ 0
--RLC
 Text HLabel 14950 9250 2    50   BiDi ~ 0
 -RLC
@@
 +RLC
 Wire Wire Line
-	14800 9050 14800 9100
-Wire Wire Line
-	14800 9100 14800 9250
-Connection ~ 14800 9100
-Wire Wire Line
-	14800 9100 14950 9100
-Wire Wire Line
 	14950 8650 14800 8650
 Connection ~ 14800 8650
@@
 	0    -1   -1   0
 $EndComp
-Text Notes 15350 9000 0    50   ~ 0
-To protector\nrelay coil
-Wire Notes Line
-	15300 8800 15300 9050
-Wire Notes Line
-	15300 9050 15850 9050
-Wire Notes Line
-	15850 9050 15850 8800
-Wire Notes Line
-	15850 8800 15300 8800
 $Comp
 L VCGA:RESISTOR R702
@@
 Text GLabel 14200 1750 2    50   BiDi ~ 0
 M_VSWON
-Text Notes 15350 8200 0    50   ~ 0
-To protector\nrelay +NC
+Text Notes 15250 9600 0    50   ~ 0
+To SPEAKER\nTERMINAL (+)
 Wire Notes Line
-	15300 8000 15300 8250
+	15200 9400 15200 9650
 Wire Notes Line
-	15300 8250 15850 8250
+	15200 9650 15850 9650
 Wire Notes Line
-	15850 8250 15850 8000
+	15850 9650 15850 9400
 Wire Notes Line
-	15850 8000 15300 8000
+	15850 9400 15200 9400
 $Comp
 L VCGA:RESISTOR R520
@@
 Wire Wire Line
 	15750 4000 15800 4000
-Wire Wire Line
-	15800 4000 15800 4900
 $Comp
 L VCGA:DIODE D701
@@
 	15150 4000 15300 4000
 Wire Wire Line
-	15800 4900 15700 4900
-Wire Wire Line
-	15800 4900 15800 7650
-Wire Wire Line
-	15800 7650 15400 7650
-Wire Wire Line
-	15400 7650 15400 7900
-Wire Wire Line
-	15400 7900 15550 7900
-Connection ~ 15800 4900
-Wire Wire Line
 	15000 7650 12450 7650
 Wire Wire Line
@@
 Wire Wire Line
 	5100 6900 5100 7350
+$Comp
+L VCGA:RELAY_STD SR701
+U 1 1 5CF04984
+P 15200 8950
+F 0 "SR701" H 15500 8950 50  0000 L CNN
+F 1 "sw1 ON" H 15480 8912 40  0001 L CNN
+F 2 "VCGA:RL-SLA24" H 15200 8950 40  0001 C CNN
+F 3 "" H 15200 8950 40  0001 C CNN
+	1    15200 8950
+	1    0    0    -1
+$EndComp
+Wire Wire Line
+	14800 8650 14800 8750
+Wire Wire Line
+	14800 9050 14800 9150
+Wire Wire Line
+	14800 8750 15100 8750
+Wire Wire Line
+	15100 8750 15100 8800
+Connection ~ 14800 8750
+Wire Wire Line
+	14800 8750 14800 8850
+Wire Wire Line
+	15100 9100 15100 9150
+Wire Wire Line
+	15100 9150 14800 9150
+Connection ~ 14800 9150
+Wire Wire Line
+	14800 9150 14800 9250
+Wire Wire Line
+	15550 9300 15300 9300
+Wire Wire Line
+	15300 9300 15300 9150
+Wire Wire Line
+	15300 8800 15300 8050
+Wire Wire Line
+	15300 7650 15800 7650
+Wire Wire Line
+	15800 4000 15800 7650
+Wire Wire Line
+	15450 9150 15300 9150
+Connection ~ 15300 9150
+Wire Wire Line
+	15300 9150 15300 9100
+$Comp
+L VCGA:RESISTOR R720
+U 1 1 5D048A7D
+P 15450 8250
+F 0 "R720" H 15600 8350 50  0000 C CNN
+F 1 "100k" H 15600 8250 50  0000 C CNN
+F 2 "VCGA:RESISTOR_AXIAL_0.5W" H 15450 8250 50  0001 C CNN
+F 3 "" H 15450 8250 50  0001 C CNN
+F 4 "0.5W" H 15600 8150 50  0000 C CNN "Wattage"
+	1    15450 8250
+	1    0    0    -1
+$EndComp
+$Comp
+L pspice:0 #GND?
+U 1 1 5D04E441
+P 15450 8450
+F 0 "#GND?" H 15450 8350 50  0001 C CNN
+F 1 "0" H 15450 8537 50  0001 C CNN
+F 2 "" H 15450 8450 50  0001 C CNN
+F 3 "~" H 15450 8450 50  0001 C CNN
+	1    15450 8450
+	1    0    0    -1
+$EndComp
+Wire Wire Line
+	15450 8400 15450 8450
+Wire Wire Line
+	15450 8100 15450 8050
+Wire Wire Line
+	15450 8050 15300 8050
+Connection ~ 15300 8050
+Wire Wire Line
+	15300 8050 15300 7650
 $EndSCHEMATC

Commit message: Commit Wed May 15 20:44:50 UTC 2019
Parts:
- SR701: Specification (none) -> SLA-24VDC-S L-C
Other:
- note added: "To OUTPUT\nTERMINAL (+)"
- note removed: "To SPEAKER\nTERMINAL (+)"
Changed lines of the file:
@@
 EESchema Schematic File Version 4
-LIBS:ANALYSIS-1500WRMS-VCGA-CLASS-H-AUDIO-POWER-AMPLIFIER-NS-LAB-VERSION-cache
+LIBS:1500WRMS-VCGA-CLASS-H-AUDIO-POWER-AMPLIFIER-NS-LAB-VERSION-cache
 EELAYER 29 0
 EELAYER END
 $Descr A3 16535 11693
 encoding utf-8
-Sheet 2 2
+Sheet 1 1
 Title "1500W RMS Class-H Audio Power Amplifier Core Circuit"
-Date "2019-05-13"
+Date "2019-05-15"
 Rev ""
 Comp "Copyright (C) Heru Himawan Tejo Laksono. All rights reserved."
@@
 M_VSWON
 Text Notes 15250 9600 0    50   ~ 0
-To SPEAKER\nTERMINAL (+)
+To OUTPUT\nTERMINAL (+)
 Wire Notes Line
 	15200 9400 15200 9650
@@
 F 2 "VCGA:RL-SLA24" H 15200 8950 40  0001 C CNN
 F 3 "" H 15200 8950 40  0001 C CNN
+F 4 "SLA-24VDC-S L-C" H 15600 9100 35  0000 C CNB "Specification"
 	1    15200 8950
 	1    0    0    -1
