File: schematics/1500WRMS-VCGA-CLASS-H-AUDIO-POWER-AMPLIFIER-NS-LAB-VERSION/ANALYSIS-1500WRMS-VCGA-CLASS-H-AUDIO-POWER-AMPLIFIER-NS-LAB-VERSION.sch (KiCad schematic (older format))
At the start: 6 parts

Commit message: Commit Wed May  8 11:35:14 UTC 2019
Parts:
- added Rdummy2: 660, symbol VCGA:RESISTOR
- added Rdummy3: 100k, symbol VCGA:RESISTOR
- added SR701: sw1 ON, symbol VCGA:RELAY_STD
- added V6, V7: 15V DC, symbol pspice:VSOURCE
Connections:
- net labels added: +120V, +15V, +42V, +RLC, -120V, -15V, -42V, -RLC, M_OUT, M_SP
- net labels removed: M_VCCHN, M_VCCHP, M_VCCLN, M_VCCLP
- wire segments 25 -> 51
Other:
- moved on the sheet: Rdummy1, V1, V2, V3, V4, V5

Commit message: Commit Wed May 15 20:03:55 UTC 2019
Parts:
- removed Rdummy3: 100k, symbol VCGA:RESISTOR
- removed SR701: sw1 ON, symbol VCGA:RELAY_STD
Connections:
- net labels removed: M_SP
- wire segments 51 -> 42
Other:
- moved on the sheet: Rdummy1
Changed lines of the file:
@@
 L pspice:0 #GND0107
 U 1 1 5C87D2BC
-P 8150 6050
-F 0 "#GND0107" H 8150 5950 50  0001 C CNN
-F 1 "0" H 8150 6140 50  0001 C CNN
-F 2 "" H 8150 6050 50  0001 C CNN
-F 3 "~" H 8150 6050 50  0001 C CNN
-	1    8150 6050
+P 9500 4350
+F 0 "#GND0107" H 9500 4250 50  0001 C CNN
+F 1 "0" H 9500 4440 50  0001 C CNN
+F 2 "" H 9500 4350 50  0001 C CNN
+F 3 "~" H 9500 4350 50  0001 C CNN
+	1    9500 4350
 	1    0    0    -1
 $EndComp
-Wire Wire Line
-	7700 3900 7300 3900
 Text Label 7400 3350 0    40   ~ 0
 +RLC
@@
 M_OUT
 Wire Wire Line
-	8150 6000 8150 6050
-Text Label 8150 5650 0    40   ~ 0
-M_SP
-Wire Wire Line
-	7950 5550 7950 5750
-Wire Wire Line
-	7950 5750 7350 5750
-Wire Wire Line
-	7950 5250 7950 5200
-Wire Wire Line
-	7950 5200 7350 5200
-Wire Wire Line
-	8150 5250 8150 5200
-Text Label 7500 5200 0    40   ~ 0
-+RLC
-Text Label 7500 5750 0    40   ~ 0
--RLC
-Text Label 8350 5200 0    40   ~ 0
-M_OUT
-Wire Wire Line
-	8150 5200 8800 5200
-Wire Wire Line
-	8800 5250 8800 5200
-Connection ~ 8800 5200
-Wire Wire Line
-	8800 5200 9050 5200
-Wire Wire Line
-	8800 5550 8800 5650
-Wire Wire Line
-	8150 5550 8150 5700
-$Comp
-L pspice:0 #GND0126
-U 1 1 6CFFF740
-P 8800 5650
-F 0 "#GND0126" H 8800 5550 50  0001 C CNN
-F 1 "0" H 8800 5740 50  0001 C CNN
-F 2 "" H 8800 5650 50  0001 C CNN
-F 3 "~" H 8800 5650 50  0001 C CNN
-	1    8800 5650
-	1    0    0    -1
-$EndComp
-$Comp
-L VCGA:RESISTOR Rdummy3
-U 1 1 69DEA6D1
-P 8800 5400
-F 0 "Rdummy3" H 8855 5447 50  0000 L CNN
-F 1 "100k" H 8855 5354 50  0000 L CNN
-F 2 "" H 8800 5400 50  0001 C CNN
-F 3 "" H 8800 5400 50  0001 C CNN
-	1    8800 5400
-	1    0    0    -1
-$EndComp
+	9500 4300 9500 4350
 $Comp
 L VCGA:RESISTOR Rdummy1
 U 1 1 5C87D0DC
-P 8150 5850
-F 0 "Rdummy1" H 8205 5897 50  0000 L CNN
-F 1 "4" H 8205 5804 50  0000 L CNN
-F 2 "" H 8150 5850 50  0001 C CNN
-F 3 "" H 8150 5850 50  0001 C CNN
-	1    8150 5850
-	1    0    0    -1
-$EndComp
-$Comp
-L VCGA:RELAY_STD SR701
-U 1 1 69DE1F65
-P 8050 5400
-F 0 "SR701" H 8331 5439 40  0000 L CNN
-F 1 "sw1 ON" H 8331 5362 40  0000 L CNN
-F 2 "" H 8050 5400 40  0001 C CNN
-F 3 "" H 8050 5400 40  0001 C CNN
-	1    8050 5400
+P 9500 4150
+F 0 "Rdummy1" H 9555 4197 50  0000 L CNN
+F 1 "4" H 9555 4104 50  0000 L CNN
+F 2 "" H 9500 4150 50  0001 C CNN
+F 3 "" H 9500 4150 50  0001 C CNN
+	1    9500 4150
 	1    0    0    -1
 $EndComp
@@
 	1    0    0    -1
 $EndComp
+Wire Wire Line
+	9500 3900 9500 4000
+Wire Wire Line
+	7300 3900 9500 3900
 $EndSCHEMATC
