File: schematics/1500WRMS-VCGA-CLASS-H-AUDIO-POWER-AMPLIFIER-NS-LAB-VERSION/1500WRMS-VCGA-CLASS-H-AUDIO-POWER-AMPLIFIER-NS-LAB-VERSION.kicad_pcb (KiCad board)
At the start: 2 copper layers, 267 parts, among them Q301 2N5551, Q401 2N5551, Q402 2N5551, Q403 2N5551, Q404 MJE340, Q405 MJE350, Q406 MJE350, Q407 MJE350, Q408 2N5551, Q409 MJE340, Q501 2N5401, Q502 MJE350, Q503 2N5551, Q504 MJE340, Q505 MJE340, Q506 MJE15032, Q507 2SC5200, Q5081 2SC5200, Q50810 2SC5200, Q50811 2SC5200, Q5082 2SC5200, Q5083 2SC5200, Q5084 2SC5200, Q5085 2SC5200, Q5086 2SC5200, Q5087 2SC5200, Q5088 2SC5200, Q5089 2SC5200, Q509 MJE15033, Q510 2SA1943, Q511 2SA1943, Q5111 2SA1943, Q51110 2SA1943, Q51111 2SA1943, Q5113 2SA1943, Q5114 2SA1943, Q5115 2SA1943, Q5116 2SA1943, Q5117 2SA1943, Q5118 2SA1943, Q5119 2SA1943, Q512 2N5551, Q513 2N5401, Q601 2N5551, Q602 2N5401, Q603 2N5401, Q604 2N5401, Q605 2N5551, Q606 2N5551, Q701 2N5551, Q702 2N5401, Q703 2N5551, Q704 2N5551, Q705 TIP42C, X6011 IRF9540, X6012 IRF9540, X6021 IRF540, X6022 IRF540

Commit message: Commit Thu May  9 11:52:12 UTC 2019
Parts:
- removed the R619 at (173.4, 66.4)
- added R305: 100k, VCGA:RESISTOR_AXIAL_0.5W, F.Cu at (268.0, 79.8)
- added R310: 2.7k, VCGA:RESISTOR_AXIAL_0.25W, F.Cu at (265.5, 84.6)
- renumbered R305 to R309, R309 to R311, R310 to R312, R311 to R313, R312 to R314
Connections:
- C301 pad 1: M_INPUT -> (no net)
- L501 pad 2: M_OUT -> (no net)
- R309 pad 2: Net-(R305-Pad2) -> Net-(R309-Pad2)
- XU302 pad 3: Net-(R305-Pad2) -> Net-(R309-Pad2)

Commit message: Commit Mon May 13 03:19:53 UTC 2019
Parts:
- R4011: value 300 -> 330
- R605, R614, R701: footprint VCGA:RESISTOR_AXIAL_0.25W -> VCGA:RESISTOR_AXIAL_0.5W
- X6011, X6012, X6021, X6022: footprint VCGA:TO-220 -> VCGA:TO-220-MIRRORED
- moved Q401 258.3 mm to (-14.0, 66.0), turned to 90 degrees
- moved R609 243.4 mm to (279.4, 0.00)
- moved C403 242.4 mm to (-6.35, 92.7), turned to 270 degrees
- moved C402 234.3 mm to (-11.4, 80.0), turned to 90 degrees
- moved Q403 233.2 mm to (-10.2, 106.7), turned to 90 degrees
- moved R614 227.3 mm to (317.5, -8.58)
- moved R4042 226.6 mm to (-7.62, 80.0), turned to 90 degrees
- moved R605 222.0 mm to (317.5, -14.2)
- moved R4131 217.1 mm to (-1.27, 38.1), turned to 270 degrees
- moved R4132 214.8 mm to (1.27, 38.1), turned to 270 degrees
- moved Q402 213.9 mm to (-8.89, 66.0), turned to 90 degrees
- moved XRV401 208.4 mm to (-11.4, 38.1)
- moved R4051 205.8 mm to (-17.8, 38.1), turned to 270 degrees
- moved R4111 201.3 mm to (-7.62, 106.7), turned to 270 degrees
- moved R4012 199.9 mm to (-15.2, 80.0), turned to 270 degrees
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- renumbered Q511 to Q5112
Connections:
- D701 pad 1: 0 -> Net-(D701-Pad1)
- D701 pad 2: Net-(D701-Pad2) -> 0
- D702 pad 1: Net-(D701-Pad2) -> 0
- D702 pad 2: 0 -> Net-(D701-Pad1)
- R4011 pad 1: Net-(C401-Pad2) -> /M_REF
- R4011 pad 2: /M_REF -> Net-(C401-Pad2)
- R4012 pad 1: Net-(C401-Pad2) -> /M_REF
- R4012 pad 2: /M_REF -> Net-(C401-Pad2)
- R701 pad 2: Net-(D701-Pad2) -> Net-(D701-Pad1)
- XU701 pad 3: Net-(D701-Pad2) -> Net-(D701-Pad1)
Other:
- net class 120V added: clearance 0.254, trace_width 1.778, via_dia 0.889, via_drill 0.508
- net class Default: clearance 0.2 -> 0.254; trace_width 0.25 -> 0.635; via_dia 0.8 -> 0.889; via_drill 0.4 -> 0.508
- rule trace_clearance: 0.2 -> 0.254
- rule trace_min: 0.2 -> 0.254

Commit message: Commit Wed May 15 20:03:55 UTC 2019
Parts:
- moved R701 302.3 mm to (40.6, 59.7), turned to 180 degrees
- moved R5139 302.2 mm to (214.6, 109.2), turned to 210 degrees
- moved XU701 301.9 mm to (40.6, 74.9), turned to 180 degrees
- moved D702 298.3 mm to (26.7, 63.5)
- moved R51311 290.8 mm to (260.4, 109.2), turned to 210 degrees
- moved R5138 277.6 mm to (191.8, 109.2), turned to 210 degrees
- moved R5137 262.8 mm to (168.9, 109.2), turned to 210 degrees
- moved R713 261.2 mm to (54.6, 67.3)
- moved C701 260.5 mm to (26.7, 72.4), turned to 180 degrees
- moved R5151 256.9 mm to (29.2, 102.9), turned to 210 degrees
- moved R51310 255.8 mm to (237.5, 109.2), turned to 210 degrees
- moved R708 254.8 mm to (54.6, 74.9)
- moved D704 253.9 mm to (26.7, 82.5)
- moved Q702 252.7 mm to (54.6, 59.7)
- moved R5136 243.4 mm to (146.1, 109.2), turned to 210 degrees
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Other:
- net class Default: trace_width 0.635 -> 0.762

Commit message: Commit Wed May 15 20:21:28 UTC 2019
Parts:
- added R720: 100k, VCGA:RESISTOR_AXIAL_0.5W, F.Cu at (-26.4, -14.2)
- added SR701: sw1 ON, VCGA:RL-SLA24, F.Cu at (-35.3, -2.26)
Connections:
- net +RLC renamed /+RLC
- net -RLC renamed /-RLC
- L501 pad 2: (no net) -> Net-(L501-Pad2)
